Commit message: feat: add configurable industrial gripper control

File: mfja_3rd_floor_description/urdf/kuka_kr6r900sixx.urdf (robot description, URDF)
Before this commit: robot kuka_kr6r900sixx, 12 links, 11 joints
Links:
- added link gripper_left_jaw, mass 0.1; visual mesh filename=package://mfja_3rd_floor_description/models/kuka_kr6r900six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 scale=1 1 1
- added link gripper_right_jaw, mass 0.1; visual mesh filename=package://mfja_3rd_floor_description/models/kuka_kr6r900six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 scale=1 1 1
- link gripper: geometry visual box size=0.063 0.008 0.022; visual box size=0.140 0.036 0.030
Joints:
- added joint gripper_left_jaw_joint: type prismatic, parent gripper, child gripper_left_jaw, origin xyz=0 0 0 rpy=0 0 0, axis -1 0 0, limit lower=0 upper=0.030 effort=150 velocity=0.18
- added joint gripper_right_jaw_joint: type prismatic, parent gripper, child gripper_right_jaw, origin xyz=0 0 0 rpy=0 0 0, axis 1 0 0, limit lower=0 upper=0.030 effort=150 velocity=0.18

File: mfja_3rd_floor_description/urdf/staubli_tx2_60l.urdf (robot description, URDF)
Before this commit: robot staubli_tx2_60l, 12 links, 11 joints
Links:
- added link gripper_left_jaw, mass 0.04; visual box size=0.020 0.010 0.040; visual box size=0.0218 0.011 0.0099
- added link gripper_right_jaw, mass 0.04; visual box size=0.020 0.010 0.040; visual box size=0.0218 0.011 0.0099
- link gripper: geometry visual box size=0.050 0.025 0.0148; visual cylinder length=0.0225 radius=0.0375
Joints:
- added joint gripper_left_jaw_joint: type prismatic, parent gripper, child gripper_left_jaw, origin xyz=0 0 0 rpy=0 0 0, axis -1 0 0, limit lower=0 upper=0.0025 effort=100 velocity=0.17
- added joint gripper_right_jaw_joint: type prismatic, parent gripper, child gripper_right_jaw, origin xyz=0 0 0 rpy=0 0 0, axis 1 0 0, limit lower=0 upper=0.0025 effort=100 velocity=0.17

File: mfja_3rd_floor_description/urdf/yaskawa_hc10.urdf (robot description, URDF)
Before this commit: robot yaskawa_hc10, 13 links, 12 joints
Links:
- link gripper: geometry visual box size=0.072 0.042 0.004; visual box size=0.090 0.078 0.048
- link gripper_left_jaw: geometry visual box size=0.003 0.019 0.035; visual box size=0.012 0.018 0.060
- link gripper_right_jaw: geometry visual box size=0.003 0.019 0.035; visual box size=0.012 0.018 0.060
Joints:
- joint gripper_left_jaw_joint: axis (none) -> -1 0 0; limit (none) -> lower=0.0 upper=0.040 effort=80.0 velocity=0.06; type fixed -> prismatic
- joint gripper_right_jaw_joint: axis (none) -> 1 0 0; limit (none) -> lower=0.0 upper=0.040 effort=80.0 velocity=0.06; type fixed -> prismatic

File: mfja_3rd_floor_description/urdf/yaskawa_hc10dt.urdf (robot description, URDF)
Before this commit: robot yaskawa_hc10dt, 11 links, 10 joints
Links:
- added link gripper_left_jaw; visual box size=0.014 0.003 0.030; visual box size=0.016 0.018 0.045
- added link gripper_right_jaw; visual box size=0.014 0.003 0.030; visual box size=0.016 0.018 0.045
- link gripper: geometry visual box size=0.040 0.070 0.012; visual box size=0.060 0.072 0.060
Joints:
- added joint gripper_left_jaw_joint: type prismatic, parent gripper, child gripper_left_jaw, origin xyz=0 -0.025 0.1065 rpy=0 0 0, axis 0 -1 0, limit lower=0.0 upper=0.010 effort=80.0 velocity=0.08
- added joint gripper_right_jaw_joint: type prismatic, parent gripper, child gripper_right_jaw, origin xyz=0 0.025 0.1065 rpy=0 0 0, axis 0 1 0, limit lower=0.0 upper=0.010 effort=80.0 velocity=0.08
