Commit message: [room315] Prepare stable manipulation training flow
Add training assets and tests, simplify the manipulation entry points, and streamline planning and execution.

File: mfja_3rd_floor_description/urdf/staubli_tx2_60l.urdf (robot description, URDF)
Before this commit: robot staubli_tx2_60l, 12 links, 11 joints
Links:
- added link gripper_mount; collision cylinder length=0.024 radius=0.0375
- link base_link: geometry collision mesh filename=package://mfja_3rd_floor_description/models/staubli_tx2_60l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; visual mesh filename=package://mfja_3rd_floor_description/models/staubli_tx2_60l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
- link gripper: geometry collision box size=0.0232 0.01 0.0415; collision box size=0.0232 0.01 0.0415
- link link_1: geometry collision mesh filename=package://mfja_3rd_floor_description/models/staubli_tx2_60l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; visual mesh filename=package://mfja_3rd_floor_description/models/staubli_tx2_60l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
- link link_2: geometry collision mesh filename=package://mfja_3rd_floor_description/models/staubli_tx2_60l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; visual mesh filename=package://mfja_3rd_floor_description/models/staubli_tx2_60l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
- link link_3: geometry collision mesh filename=package://mfja_3rd_floor_description/models/staubli_tx2_60l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; visual mesh filename=package://mfja_3rd_floor_description/models/staubli_tx2_60l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
- link link_4: geometry collision mesh filename=package://mfja_3rd_floor_description/models/staubli_tx2_60l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; visual mesh filename=package://mfja_3rd_floor_description/models/staubli_tx2_60l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
- link link_5: geometry collision mesh filename=package://mfja_3rd_floor_description/models/staubli_tx2_60l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; visual mesh filename=package://mfja_3rd_floor_description/models/staubli_tx2_60l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
- link link_6: geometry collision mesh filename=package://mfja_3rd_floor_description/models/staubli_tx2_60l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; visual mesh filename=package://mfja_3rd_floor_description/models/staubli_tx2_60l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
Joints:
- removed joint tool0_gripper
- added joint gripper_mount_joint: type fixed, parent gripper_mount, child gripper, origin xyz=0 0 0 rpy=0 0 0
- added joint tool0_gripper_mount_joint: type fixed, parent tool0, child gripper_mount, origin xyz=0 0 0 rpy=0 0 0

File: mfja_staubli_manipulation_demos/hpp/room315_shuttle_deck.urdf (robot description, URDF)
Before this commit: robot room315_shuttle_deck, 1 links, 0 joints
Links:
- link deck_link: geometry collision box size=0.36 0.22 0.17; visual box size=0.36 0.22 0.17

File: mfja_staubli_manipulation_demos/hpp/room315_staubli_table_drop_zone.urdf (robot description, URDF)
Before this commit: robot room315_staubli_table_drop_zone, 1 links, 0 joints
Links:
- link drop_zone_link: geometry collision mesh filename=package://mfja_3rd_floor_description/models/staubli_table/m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; visual box size=0.36 0.24 0.02
