Commit message: [room315] Add portable table pick-and-place

File: mfja_3rd_floor_description/urdf/room315_cell.urdf (robot description, URDF)
Before this commit: robot room315_cell, 7 links, 6 joints
Links:
- added link room_shell; visual mesh filename=package://mfja_3rd_floor_description/models/room_315/meshes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
- link carter_droit: geometry collision mesh filename=package://mfja_3rd_floor_description/models/carter_droit/me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; visual mesh filename=package://mfja_3rd_floor_description/models/carter_droit/me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
- link carter_gauche: geometry collision mesh filename=package://mfja_3rd_floor_description/models/carter_gauche/m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; visual mesh filename=package://mfja_3rd_floor_description/models/carter_gauche/m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
- link cell_path_left: geometry collision mesh filename=package://mfja_3rd_floor_description/models/cell_path_left/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; visual mesh filename=package://mfja_3rd_floor_description/models/cell_path_left/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
- link cell_path_right: geometry collision mesh filename=package://mfja_3rd_floor_description/models/cell_path_right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; visual mesh filename=package://mfja_3rd_floor_description/models/cell_path_right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
- link cell_static_droit: geometry collision mesh filename=package://mfja_3rd_floor_description/models/cell_static_dro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; visual mesh filename=package://mfja_3rd_floor_description/models/cell_static_dro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
- link cell_static_gauche: geometry collision mesh filename=package://mfja_3rd_floor_description/models/cell_static_gau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; visual mesh filename=package://mfja_3rd_floor_description/models/cell_static_gau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
Joints:
- added joint room_shell_joint: type fixed, parent base, child room_shell, origin xyz=0 0 0 rpy=0 0 -1.57
- joint cell_path_left_joint: origin xyz=-11.865 -5.56 0.733 rpy=0 0 0 -> xyz=-11.865 -5.56 1.05 rpy=0 0 0
- joint cell_path_right_joint: origin xyz=-13.705 -3.843 0.733 rpy=0 0 3.14 -> xyz=-13.705 -3.843 1.05 rpy=0 0 3.14
- joint cell_static_droit_joint: origin xyz=-15.9170 -5.81 0 rpy=0 0 0 -> xyz=-15.9170 -5.81 0.317 rpy=0 0 0
- joint cell_static_gauche_joint: origin xyz=-9.65 -3.6 0 rpy=0 0 3.14 -> xyz=-9.65 -3.6 0.317 rpy=0 0 3.14

File: mfja_staubli_manipulation_demos/hpp/room315_staubli_table_drop_zone.urdf (robot description, URDF)
Before this commit: robot room315_staubli_table_drop_zone, 1 links, 0 joints
Links:
- link drop_zone_link: geometry collision mesh filename=package://mfja_3rd_floor_description/models/staubli_table/m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; visual box size=0.36 0.24 0.02
